File: Atari OSS Cartridge.kicad_pcb (KiCad board)
At the start: 2 copper layers, 39 x 32.2 mm, 23 parts, among them J1 Basic_a, J2 Basic_b, J3 A14_16_sel, J4 on_off, J6 OUT_SIGNAL, U1 27C010, U2 74LS74, U3 74HC02, U4 74HC02, U5 74LS157

Commit message: Tracking
Parts:
- added C8: 100n, Capacitor_SMD:C_0603_1608Metric_Pad1.05x0.95mm_HandSolder, F.Cu at (125.1, 101.1)
- moved J6 20.1 mm to (119.1, 114.8), turned to 270 degrees
- moved U3 11.4 mm to (123.1, 95.3)
- moved C7 8.26 mm to (125.1, 89.6)
- moved C1 5.66 mm to (115.9, 89.6)
- moved U2 5.58 mm to (113.8, 95.3)
- moved C2 5.38 mm to (115.9, 101.1)
- moved U4 5.38 mm to (113.8, 106.7)
- moved C5 4.29 mm to (115.9, 87.1), turned to 180 degrees
- moved J4 3.35 mm to (122.8, 114.8)
- moved C6 3.20 mm to (124.2, 86.9), turned to 0 degrees
- moved U5 3.09 mm to (123.1, 107.2)
Routing:
- net A12: track 12.5 -> 51.1 mm, vias 1 -> 6
- net Net-(U1-Pad28): track 0.00 -> 35.5 mm, vias 0 -> 3
- net Net-(U1-Pad4): track 0.00 -> 32.6 mm, vias 0 -> 2
- net Net-(U4-Pad1): track 1.72 -> 31.6 mm, vias 1 -> 2
- net Net-(J4-Pad1): track 0.00 -> 27.8 mm, vias 0 -> 3
- net CCTL: track 0.00 -> 26.8 mm, vias 0 -> 3
- net O2: track 1.27 -> 25.2 mm, vias 0 -> 2
- net Net-(U1-Pad22): track 2.54 -> 25.7 mm
- net RD5_OUT: track 0.00 -> 21.3 mm
- net A14_SEL: track 0.00 -> 19.7 mm
- net Net-(U3-Pad4): track 1.59 -> 17.6 mm, vias 1 -> 2
- net A15_SEL: track 0.00 -> 15.5 mm
- net Net-(U2-Pad11): track 21.3 -> 5.93 mm, vias 2 -> 0
- net VCC: track 100.0 -> 85.0 mm, vias 9 -> 1
- net A16_SEL: track 0.00 -> 14.0 mm
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Other:
- board text removed: "74HC02"
- board text removed: "74HC74"
- board text removed: "74LHC02"
- board text removed: "A12"
- board text removed: "A13"
- board text removed: "Basic"
- board text removed: "S5"

Commit message: Tracking
Parts:
- moved R5 31.4 mm to (111.8, 89.6), turned to 180 degrees
- moved R6 26.5 mm to (121.0, 101.1), turned to 180 degrees
- moved C5 0.34 mm to (115.6, 86.9)
- moved C6 0.16 mm to (124.1, 87.1)
Routing:
- net Net-(R5-Pad1): track 0.00 -> 49.2 mm, vias 0 -> 2
- net A0: track 6.47 -> 49.3 mm, vias 0 -> 1
- net GND: track 142.3 -> 99.9 mm, vias 7 -> 21
- net VCC: track 85.0 -> 114.4 mm
- net A3: track 11.8 -> 36.8 mm, vias 0 -> 2
- net Net-(C6-Pad1): track 5.93 -> 18.0 mm, vias 0 -> 2
- net Net-(U2-Pad11): track 5.93 -> 17.8 mm, vias 0 -> 2
- net Net-(U4-Pad1): track 31.6 -> 27.4 mm
- net A12: track 51.1 -> 54.7 mm, vias 6 -> 5
- net Net-(U4-Pad10): track 13.0 -> 10.6 mm
- net CCTL: track 26.8 -> 24.7 mm
- net Net-(J4-Pad1): track 27.8 -> 29.8 mm
- net RD5_OUT: track 21.3 -> 22.8 mm
- net O2: track 25.2 -> 26.6 mm
- added copper zone on B.Cu, net GND
- added copper zone on F.Cu, net GND
Other:
- board text added: "74HCT02"
- board text added: "74HCT157"
- board text added: "74HCT74"
- board text added: "A14"
- board text added: "A15"
- board text added: "A16"
- board text added: "CCTL"
- board text added: "O2"
- board text added: "RD5"
- board text added: "S5"
- board text added: "on"

Commit message: tracking
Routing:
- net GND: track 99.9 -> 96.8 mm
- net BASIC: track 44.5 -> 45.5 mm
